File: smd-proto.sch (EAGLE design)
At the start: 65 parts

Commit message: Added bunch of boards and outline
Parts:
- removed C10, C11, C12, C13, C14, C15, C16, C17, C18, C19, C20, C21, C3, C4, C5, C6, C7, C8, C9: 0.5PF 50V, Seeed-OPL-Capacitor:CERAMIC-0.5PF-50V-0.1PF-NPO(0603)
- removed C22, C23, C24, C25, C26, C27, C28, C29, C30, C31, C32, C33, C34, C35, C36, C37, C38, C39, C40: 2.2uf, Seeed-OPL-Capacitor:CERAMIC-2.2UF-25V-10%-X7R(0805)
- added C41, C43, C45: 0.5PF 50V, Seeed-OPL-Capacitor:CERAMIC-0.5PF-50V-0.1PF-NPO(0603)
- added C42, C44, C46: 2.2uf, Seeed-OPL-Capacitor:CERAMIC-2.2UF-25V-10%-X7R(0805)
- added D1, D2: RED-0805, Seeed-OPL-Diode:SMD-LED-CLEAR-RED(0805)
- added J1: GREEN-3P-5.0, Seeed-OPL-Connector:SCREW-TERMINAL-GREEN(3P-5.0)
- added JP15, JP17, JP19, JP20, JP27: (no value), SparkFun-Connectors:M02PTH
- added JP16: (no value), SparkFun-Connectors:M09
- added JP18: FTDI_BASICPTH, SparkFun-Connectors:FTDI_BASICPTH
- added JP22, JP23, JP24, JP26, JP30, JP31: (no value), SparkFun-Connectors:M08NO_SILK_FEMALE_PTH
- added K1, K2: TS-1109-7, Seeed-OPL-Switch:DIP-BUTTON-TOP-BLACK(4P-D6.2MM)
- added R1, R3: 1.1M 1/10W, Seeed-OPL-Resistor:SMD-RES-1.1M-1%-1/10W(0603)
- added R2: 1K, Seeed-OPL-Resistor:SMD-RES-5.6K-5%-1/10W(0603)
- added U1: ATMEGA328P_PDIP, SparkFun-DigitalIC:ATMEGA328P_PDIP
- added Y1: 16MHZ, Seeed-OPL-crystal-osctllator:SMD-CRYSTAL-16MHZ-8PF-20PPM-40R(2P-5.0X3.2MM)
- C1: value 0.5PF 50V -> 22pf; device Seeed-OPL-Capacitor:CERAMIC-0.5PF-50V-0.1PF-NPO(0603) -> Seeed-OPL-Capacitor:CERAMIC-22PF-50V-5%-NPO(0603)
- C2: value 2.2uf -> 22pf; device Seeed-OPL-Capacitor:CERAMIC-2.2UF-25V-10%-X7R(0805) -> Seeed-OPL-Capacitor:CERAMIC-22PF-50V-5%-NPO(0603)
- JP10, JP9: device SparkFun-Connectors:M01NOSILK-KIT -> SparkFun-Connectors:M14
- JP11: device SparkFun-Connectors:M01NOSILK-KIT -> SparkFun-Connectors:DB9MALE
- JP12: device SparkFun-Connectors:M01NOSILK-KIT -> SparkFun-Connectors:M09
- JP13: device SparkFun-Connectors:M01NOSILK-KIT -> SparkFun-Connectors:DB9FEMALE
- JP4, JP6: device SparkFun-Connectors:M01NOSILK-KIT -> SparkFun-Connectors:M02PTH
- JP5: device SparkFun-Connectors:M01NOSILK-KIT -> SparkFun-Connectors:M03PTH
- JP7: value (none) -> RJ45; device SparkFun-Connectors:M01NOSILK-KIT -> SparkFun-Connectors:RJ45-8PTH
- JP8: device SparkFun-Connectors:M01NOSILK-KIT -> SparkFun-Connectors:M08
Connections:
- removed net N$100: C35.2, C36.1
- removed net N$102: C18.1, C37.1, JP12.1
- removed net N$96: C13.2, C36.2, JP11.1
- removed net N$98: C33.2, C34.1
- removed net N$99: C34.2, C35.1
- new net A_A0: JP9.6, U1.PC0(ADC0)
- new net A_A1: JP9.5, U1.PC1(ADC1)
- new net A_A2: JP9.4, U1.PC2(ADC2)
- new net A_A3: JP9.3, U1.PC3(ADC3)
- new net A_A4/SDC: JP9.2, U1.PC4(ADC4/SDA)
- new net A_A5/SCL: JP9.1, U1.PC5(ADC5/SCL)
- new net A_AREF: JP10.13, U1.AREF
- new net A_D0/RX: JP10.4, U1.PD0(RXD)
- new net A_D1/TX: JP10.5, U1.PD1(TXD)
- new net A_D10~: JP9.13, U1.PB2(SS/OC1B)
- new net A_D11~/MOSI: JP9.12, U1.PB3(MOSI/OC2)
- new net A_D2: JP10.6, U1.PD2(INT0)
- new net A_D3~: JP10.7, U1.PD3(INT1)
- new net A_D4: JP10.8, U1.PD4(XCK/T0)
- new net A_D5~: JP10.9, U1.PD5(T1)
- new net A_D6~: JP10.10, U1.PD6(AIN0)
- new net A_D7: JP10.11, U1.PD7(AIN1)
- new net A_D8: JP10.12, U1.PB0(ICP)
- new net A_D9~: JP10.14, JP9.14, U1.PB1(OC1A)
- new net A_GND: C1.1, C2.1, JP10.2, JP9.9, U1.GND@1, U1.GND@2
- new net A_RESET: JP10.3, R2.2, U1.PC6(/RESET)
- new net A_VCC: JP10.1, JP9.8, R2.1, U1.AVCC, U1.VCC
- new net D12/MISO: JP9.11, U1.PB4(MISO)
- new net D13/SCK: JP9.10, U1.PB5(SCK)
- new net FTDI_CTS: JP18.5
- new net FTDI_DTR: JP18.1
- new net FTDI_GND: JP18.6
- new net FTDI_RX: JP18.2
- new net FTDI_TX: JP18.3
- new net FTDI_VCC: JP18.4
- new net N$108: JP27.2, R3.2
- new net N$43: C41.1, C42.1, JP15.1
- new net N$44: C41.2, C42.2, JP15.2
- new net N$45: C43.1, C44.1, JP17.1
- new net N$46: C43.2, C44.2, JP17.2
- new net N$47: C45.1, C46.1, JP19.1
- new net N$50: C45.2, C46.2, JP19.2
- new net N$52: JP4.2, K1.A0, K1.A1
- new net N$55: D1.+, JP6.1
- new net N$56: D1.-, R1.1
- new net N$76: JP11.1, JP12.1
- new net N$92: JP13.6, JP16.6
- net N$103: now also JP20.1, K2.B0, K2.B1; no longer C37.2, C38.1
- net N$104: now also JP20.2, K2.A0, K2.A1; no longer C38.2, C39.1
- net N$105: now also D2.+, JP27.1; no longer C39.2, C40.1
- net N$106: now also D2.-, R3.1; no longer C21.2, C40.2, JP13.1
- net N$41: now also JP4.1, K1.B0, K1.B1; no longer C3.2, C4.1
- net N$58: now also JP6.2, R1.2; no longer C4.2, C5.1
- net N$60: now also J1.P$2, JP5.2; no longer C1.2, C3.1
- net N$61: now also J1.P$1, JP5.1; no longer C10.1, C33.1, JP10.1
- net N$62: now also J1.P$3, JP5.3; no longer C6.2, C7.1
- net N$63: now also JP7.1, JP8.8; no longer C7.2, C8.1
- net N$64: now also JP7.2, JP8.7; no longer C8.2, C9.1
- net N$65: now also JP7.3, JP8.6; no longer C14.1, C29.1, JP8.1
- net N$66: now also JP7.4, JP8.5; no longer C17.2, C32.2, JP9.1
- net N$67: now also JP7.5, JP8.4; no longer C10.2, C11.1
- net N$68: now also JP7.6, JP8.3; no longer C11.2, C12.1
- net N$69: now also JP7.7, JP8.2; no longer C12.2, C13.1
- net N$72: now also JP7.8, JP8.1; no longer C14.2, C15.1
- net N$73: now also C1.2, U1.PB6(XTAL1/TOSC1), Y1.2; no longer C15.2, C16.1
- net N$74: now also C2.2, U1.PB7(XTAL2/TOSC2), Y1.1; no longer C16.2, C17.1
- net N$77: now also JP11.2, JP12.2; no longer C18.2, C19.1
- net N$78: now also JP11.3, JP12.3; no longer C19.2, C20.1
- net N$79: now also JP11.4, JP12.4; no longer C20.2, C21.1
- net N$82: now also JP11.5, JP12.5; no longer C1.1, C2.1, JP4.1
- net N$83: now also JP11.6, JP12.6; no longer C2.2, C22.1
- net N$84: now also JP11.7, JP12.7; no longer C22.2, C23.1
- net N$85: now also JP11.8, JP12.8; no longer C23.2, C24.1
- net N$86: now also JP11.9, JP12.9; no longer C24.2, C5.2, JP5.1
- net N$87: now also JP13.1, JP16.1; no longer C25.1, C6.1, JP6.1
- net N$88: now also JP13.2, JP16.2; no longer C25.2, C26.1
- net N$89: now also JP13.3, JP16.3; no longer C26.2, C27.1
- net N$90: now also JP13.4, JP16.4; no longer C27.2, C28.1
- net N$91: now also JP13.5, JP16.5; no longer C28.2, C9.2, JP7.1
- net N$93: now also JP13.7, JP16.7; no longer C29.2, C30.1
- net N$94: now also JP13.8, JP16.8; no longer C30.2, C31.1
- net N$95: now also JP13.9, JP16.9; no longer C31.2, C32.1
Other:
- note added: "0603/0805 breakout"
- note added: "AVR-ISP POGO PINS"
- note added: "DB9 Female breakout"
- note added: "DB9 Male breakout"
- note added: "LDO SOT223 breakout"
- note added: "LED breakout"
- note added: "Pushbutton breakout"
- note added: "SOIC16/SSOP16 breakout"
- note added: "SOT-23/SOT-89 breakout"
- note added: "SOT23-5 breakout"
- note added: "Screw terminals breakout"
- moved on the sheet: C1, C2, JP1, JP14, JP2, JP21, JP25, JP3, SOT-89, SOT223, SOT23, SOT23-5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

Commit message: Fixed ERC and DRC issues, finalized some boards
Connections:
- net A_GND: now also JP9.8
- net A_VCC: now also JP9.7; no longer JP9.8
Other:
- note added: "Minimal arduino"
- note added: "Protoboard"
- note added: "TQFP breakout"
- moved on the sheet: JP2, JP20, JP22, JP23, JP24, JP26, JP3, JP30, JP31, JP4, K1, K2
